File: mfm-micro.sch (KiCad schematic (older format))
At the start: 53 parts

Commit message: Update
Parts:
- removed J?: SPI1_connector, symbol Connector_Generic:Conn_02x03_Odd_Even
- removed J?: SPI2_connector, symbol Connector_Generic:Conn_02x03_Odd_Even
- removed J?: SPI3_connector, symbol Connector_Generic:Conn_02x03_Odd_Even
- removed R?: 1k, symbol Device:R_Small
- removed R? (x3): 10k, symbol Device:R_Small
- removed U?: STM32F070CBTx, Package_QFP:LQFP-48_7x7mm_P0.5mm, symbol MCU_ST_STM32F0:STM32F070CBTx
- added C16: 100n, Capacitor_SMD:C_0402_1005Metric, symbol Device:C_Small
- added C17: 100nf, symbol Device:C_Small
- added F1: Fuse_Small, Fuse:Fuse_0805_2012Metric, symbol Device:Fuse_Small
- added H1, H2: MountingHole_Pad, MountingHole:MountingHole_3.2mm_M3_Pad_Via, symbol Mechanical:MountingHole_Pad
- added J3: Peripheral1_connector, symbol Connector_Generic:Conn_02x04_Odd_Even
- added J5: Peripheral2_connector, symbol Connector_Generic:Conn_02x04_Odd_Even
- added J6: Peripheral3_connector, symbol Connector_Generic:Conn_02x04_Odd_Even
- added J8: UART_Connector, symbol Connector_Generic:Conn_01x06
- added R11, R12, R14: 10k, Resistor_SMD:R_0402_1005Metric, symbol Device:R_Small
- added R15, R17, R18, R19, R20, R21, R22: 130, Resistor_SMD:R_0402_1005Metric, symbol Device:R_Small
- added R16: 680, Resistor_SMD:R_0402_1005Metric, symbol Device:R_Small
- added SW3: STAT_LED_Switch, Connector_PinHeader_2.54mm:PinHeader_1x02_P2.54mm_Vertical, symbol Switch:SW_SPST
- added SW4: SW_RST, Button_Switch_THT:SW_PUSH_6mm, symbol Switch:SW_SPST
- added U4: STM32L072CBTx, Package_QFP:LQFP-48_7x7mm_P0.5mm, symbol MCU_ST_STM32L0:STM32L072CBTx
- C1, C11, C14, C15, C2, C3, C6, C7, C8, C9: renamed from C?; footprint (none) -> Capacitor_SMD:C_0402_1005Metric
- C10: renamed from C?; value 10n -> 100n; footprint (none) -> Capacitor_SMD:C_0402_1005Metric
- C12, C13: renamed from C?; value 21p -> 20p; footprint (none) -> Capacitor_SMD:C_0402_1005Metric
- C4: renamed from C?; footprint (none) -> Capacitor_SMD:C_0805_2012Metric
- C5: renamed from C?; value 4.7u -> 10u; footprint (none) -> Capacitor_SMD:C_0402_1005Metric
- D1, D4: renamed from D?; footprint (none) -> Diode_SMD:D_SOD-123
- D2, D3, D5, D6: renamed from D?; footprint (none) -> LED_SMD:LED_0603_1608Metric
- FB1, FB2: renamed from FB?; footprint (none) -> Inductor_SMD:L_0805_2012Metric
- J2: renamed from J?; footprint (none) -> Connector_JST:JST_PH_B3B-PH-K_1x03_P2.00mm_Vertical
- J4: renamed from J?; value 01x05 -> SWD_connector; footprint (none) -> Connector_PinHeader_2.54mm:PinHeader_1x05_P2.54mm_Vertical
- R1: renamed from R?; footprint (none) -> Resistor_SMD:R_1206_3216Metric
- R10, R2, R4, R6, R7, R8, R9: renamed from R?; footprint (none) -> Resistor_SMD:R_0402_1005Metric
- R13: renamed from R?; value 1k -> 130; footprint (none) -> Resistor_SMD:R_0402_1005Metric
- R3, R5: renamed from R?; value ? -> 1k; footprint (none) -> Resistor_SMD:R_0402_1005Metric
- SW1: renamed from SW?; footprint (none) -> Connector_PinHeader_2.54mm:PinHeader_1x03_P2.54mm_Vertical
- SW2: renamed from SW?; value ? -> PWR_LED_Switch; footprint (none) -> Connector_PinHeader_2.54mm:PinHeader_1x02_P2.54mm_Vertical
- U1: renamed from U?; footprint Package_TO_SOT_SMD:SOT-666 -> Package_TO_SOT_SMD:SOT-23-6
- U2: renamed from U??; footprint (none) -> Package_SO:SOP-8_3.9x4.9mm_P1.27mm
- XOSC1: renamed from XOSC?; footprint (none) -> Crystal:Crystal_SMD_3225-4Pin_3.2x2.5mm
- XOSC32: footprint (none) -> Crystal:Crystal_SMD_3215-2Pin_3.2x1.5mm
- gave numbers to parts that had none: 3
Connections:
- net +3.3VA: now also U4.9 (VDDA); no longer SW1.3 (C), SW2.1 (A)
- net +3V3: now also SW1.3 (C), SW2.1 (A), C16.1, J3.1 (Pin_1), J5.1 (Pin_1), J6.1 (Pin_1), R11.1, R12.1, R14.1, U4.1 (VDD), U4.24 (VDD), U4.36 (VDD_USB), U4.48 (VDD)
- net +BATT: no longer R2.1
- net -BATT: now also C16.2, H1.1, H2.1, J3.5 (Pin_5), J5.5 (Pin_5), J6.5 (Pin_5), J8.6 (Pin_6), R15.1, R17.1, R18.1, R19.1, R20.1, R21.1, R22.1, SW4.1 (A), U4.23 (VSS), U4.35 (VSS), U4.47 (VSS), U4.8 (VSSA)
- net BOOT0: now also U4.44 (BOOT0)
- net LED0: now also SW3.1 (A), U4.26 (PB13); no longer D5.2 (A)
- net NRST: now also C17.2, SW4.2 (B), U4.7 (NRST)
- net SPI_MISO: now also J3.4 (Pin_4), J5.4 (Pin_4), J6.4 (Pin_4), U4.16 (PA6)
- net SPI_MOSI: now also J3.6 (Pin_6), J5.6 (Pin_6), J6.6 (Pin_6), U4.17 (PA7)
- net SPI_SCK: now also J3.2 (Pin_2), J5.2 (Pin_2), J6.2 (Pin_2), U4.15 (PA5)
- net SPI_SS1: now also J3.3 (Pin_3), R11.2, U4.18 (PB0)
- net SPI_SS2: now also J5.3 (Pin_3), R12.2, U4.19 (PB1)
- net SPI_SS3: now also J6.3 (Pin_3), R14.2, U4.20 (PB2)
- net SWCLK: now also U4.37 (PA14)
- net SWDIO: now also U4.34 (PA13)
- net UART1_RX: now also J8.2 (Pin_2), U4.31 (PA10)
- net UART1_TX: now also J8.3 (Pin_3), U4.30 (PA9)
- net USB_DM: now also U4.32 (PA11)
- net USB_DP: now also U4.33 (PA12)
- net VBUS: now also R2.1
- net VCC: now also F1.1; no longer FB1.1
- net XOSC32_IN: now also U4.3 (PC14)
- net XOSC32_OUT: now also U4.4 (PC15)
- net XOSC_IN: now also U4.5 (PH0)
- net XOSC_OUT: now also R16.2, U4.6 (PH1); no longer C15.1, XOSC1.3
- net at D5.1 (K), R13.2: now also R17.2, R18.2, R19.2
- net at D6.1 (K): now also R15.2, R20.2, R21.2, R22.2
- new net: F1.2, FB1.1
- new net: C15.1, R16.1, XOSC1.3
- new net: D5.2 (A), SW3.2 (B)
- new net: C17.1, J8.1 (Pin_1)
- new net P_EXTI: J3.7 (Pin_7), J5.7 (Pin_7), J6.7 (Pin_7), U4.39 (PB3)
- no-connect marks 0 -> 24
Other:
- note added: "2020/09/14"
- note added: "Mounting holes"
- note added: "Multiflexmeter Micro Design"
- note added: "SS Pull up"
- note added: "Tim van Osch"
- note added: "UART_Connector"
- moved on the sheet: C10, C11, C12, C13, C14, C15, C5, C6, C7, C8, C9, D5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

Commit message: Place components on PCB
Parts:
- removed C16: 100n, Capacitor_SMD:C_0402_1005Metric, symbol Device:C_Small
- removed J6: Peripheral3_connector, symbol Connector_Generic:Conn_02x04_Odd_Even
- C17: value 100nf -> 100n; footprint (none) -> Capacitor_SMD:C_0402_1005Metric
- J1: footprint (none) -> Connector_USB:USB_Mini-B_Tensility_54-00023_Vertical_CircularHoles
- J8: footprint (none) -> Connector_PinHeader_2.54mm:PinHeader_1x06_P2.54mm_Vertical
- P1: renamed from J3; footprint (none) -> Connector_PinHeader_2.54mm:PinHeader_2x04_P2.54mm_Vertical
- P2: renamed from J5; footprint (none) -> Connector_PinHeader_2.54mm:PinHeader_2x04_P2.54mm_Vertical
- R3, R5: value 1k -> 100
Connections:
- net SPI_SS3: no longer U4.20 (PB2)
- net -BATT renamed GND
- no-connect marks 24 -> 23
Other:
- moved on the sheet: P1, P2, R11, R12, R14

Commit message: Rerout and new exports
Parts:
- removed C12, C13: 20p, Capacitor_SMD:C_0402_1005Metric, symbol Device:C_Small
- removed C17: 100n, Capacitor_SMD:C_0402_1005Metric, symbol Device:C_Small
- removed J8: UART_Connector, Connector_PinHeader_2.54mm:PinHeader_1x06_P2.54mm_Vertical, symbol Connector_Generic:Conn_01x06
- removed R14: 10k, Resistor_SMD:R_0402_1005Metric, symbol Device:R_Small
- removed SW1: SW_DPDT_x2, Connector_PinHeader_2.54mm:PinHeader_1x03_P2.54mm_Vertical, symbol Switch:SW_DPDT_x2
- removed SW3: STAT_LED_Switch, Connector_PinHeader_2.54mm:PinHeader_1x02_P2.54mm_Vertical, symbol Switch:SW_SPST
- removed XOSC32: 32.768KHz, Crystal:Crystal_SMD_3215-2Pin_3.2x1.5mm, symbol Device:Crystal_Small
- added J4: Conn_01x03, Connector_PinHeader_2.54mm:PinHeader_1x03_P2.54mm_Vertical, symbol Connector_Generic:Conn_01x03
- renumbered C3 to C1, C14 to C12, C15 to C13, C1 to C2, C2 to C3, J4 to J3, R16 to R10, R10 to R11, R17 to R12, R18 to R13, R13 to R14, R19 to R15, R15 to R16, R20 to R17, R21 to R18, R22 to R19, R11 to R20, R12 to R21, SW4 to SW1, SW2 to SW4, U3 to U1, U1 to U3
Connections:
- net GND: now also P1.3 (Pin_3), P2.3 (Pin_3), R11.2, J4.3 (Pin_3); no longer P1.5 (Pin_5), P2.5 (Pin_5)
- net LED0: now also D5.2 (A), U4.39 (PB3); no longer U4.26 (PB13)
- net P_EXTI: now also P1.5 (Pin_5), P2.5 (Pin_5), U4.26 (PB13); no longer P1.7 (Pin_7), P2.7 (Pin_7), U4.39 (PB3)
- net SPI_SS1: now also P1.8 (Pin_8); no longer P1.3 (Pin_3)
- net SPI_SS2: now also P2.8 (Pin_8); no longer P2.3 (Pin_3)
- net UART1_RX: now also J4.1 (Pin_1)
- net UART1_TX: now also J4.2 (Pin_2)
- net D+ renamed USB_CONN_D+
- net USB_CONN_D+: now also U3.3 (I/O2); no longer U3.4 (I/O2)
- net D- renamed USB_CONN_D-
- net USB_CONN_D-: now also U3.1 (I/O1); no longer U3.6 (I/O1)
- net USB_DM renamed USB_D-
- net USB_D-: now also U3.6 (I/O1); no longer U3.1 (I/O1)
- net USB_DP renamed USB_D+
- net USB_D+: now also U3.4 (I/O2); no longer U3.3 (I/O2)
- net XOSC32_IN: no longer names the net of U4.3 (PC14)
- net XOSC32_OUT: no longer names the net of U4.4 (PC15)
- no-connect marks 23 -> 24
Other:
- moved on the sheet: C1, C12, C13, C2, C3, F1, FB1, J1, R10, R20, R21, R4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
