File: hardware/mfm-micro.sch (KiCad schematic (older format))
At the start: 59 parts, among them J1 USB_B_Mini, J2 JST PH 3, J3 SWD_connector, J4 Conn_01x03, P1 Peripheral1_connector, P2 Peripheral2_connector, Q1 AO3401A, SW1 SW_RST, SW4 PWR_LED_Switch, U1 XC6206P332MR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

Commit message: Update docs
Parts:
- J1: symbol Connector:USB_B_Mini -> mfm-micro-rescue:USB_B_Mini-Connector
Changed lines of the file:
@@
 USB_CONN_D+
 $Comp
-L Connector:USB_B_Mini J1
+L mfm-micro-rescue:USB_B_Mini-Connector J1
 U 1 1 5F55AD22
 P 900 1200
